File: Hardware/v12.brd (EAGLE design)
At the start: 50 x 50 mm, 85 parts, among them IC1 LM324D, IC2 m328p, IC3 REG1117, IC4 OPA336U, J1 22-27-2081-08, J2 22-27-2031-03

Commit message: changed some values (led resistors) updated shopping list
Parts:
- DISP-R1, DISP-R2, DISP-R3, DISP-R4, DISP-R5, DISP-R6, DISP-R7, LED2-R1: value 300 -> 330
Changed lines of the file:
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@@
 <element name="DISP-Q2" library="transistor-small-signal" package="SOT23" value="IRLML2502" x="9.525" y="35.004375" rot="MR180"/>
 <element name="DISP-Q3" library="transistor-small-signal" package="SOT23" value="IRLML2502" x="13.335" y="35.004375" rot="MR180"/>
-<element name="DISP-R1" library="rcl" package="R0603" value="300" x="4.048125" y="29.289375" rot="R180"/>
-<element name="DISP-R2" library="rcl" package="R0603" value="300" x="4.048125" y="26.273125" rot="R180"/>
-<element name="DISP-R3" library="rcl" package="R0603" value="300" x="3.571875" y="20.081875" rot="MR90"/>
-<element name="DISP-R4" library="rcl" package="R0603" value="300" x="3.87985" y="21.078825" rot="R180"/>
-<element name="DISP-R5" library="rcl" package="R0603" value="300" x="3.889375" y="22.463125" rot="R180"/>
-<element name="DISP-R6" library="rcl" package="R0603" value="300" x="4.048125" y="27.78125" rot="R180"/>
-<element name="DISP-R7" library="rcl" package="R0603" value="300" x="15.875" y="33.258125" rot="R90"/>
+<element name="DISP-R1" library="rcl" package="R0603" value="330" x="4.048125" y="29.289375" rot="R180"/>
+<element name="DISP-R2" library="rcl" package="R0603" value="330" x="4.048125" y="26.273125" rot="R180"/>
+<element name="DISP-R3" library="rcl" package="R0603" value="330" x="3.571875" y="20.081875" rot="MR90"/>
+<element name="DISP-R4" library="rcl" package="R0603" value="330" x="3.87985" y="21.078825" rot="R180"/>
+<element name="DISP-R5" library="rcl" package="R0603" value="330" x="3.889375" y="22.463125" rot="R180"/>
+<element name="DISP-R6" library="rcl" package="R0603" value="330" x="4.048125" y="27.78125" rot="R180"/>
+<element name="DISP-R7" library="rcl" package="R0603" value="330" x="15.875" y="33.258125" rot="R90"/>
 <element name="DISP-R8\" library="rcl" package="R0603" value="300" x="14.605" y="17.8181" rot="R180"/>
 <element name="I2C" library="con-molex" package="6410-03" value="22-27-2031-03" x="23.8125" y="46.0375" rot="MR0">
@@
 <element name="LED1-R1" library="rcl" package="R0603" value="1k" x="36.3728" y="13.801725" rot="MR90"/>
 <element name="LED2" library="led" package="CHIP-LED0805" value="GN" x="4.098925" y="15.274925" rot="R180"/>
-<element name="LED2-R1" library="rcl" package="R0603" value="300" x="4.0513" y="11.731625" rot="R90"/>
+<element name="LED2-R1" library="rcl" package="R0603" value="330" x="4.0513" y="11.731625" rot="R90"/>
 <element name="OPAMP-C1" library="rcl" package="C0603" value="100n" x="41.481375" y="14.89075" rot="MR0"/>
 <element name="OPAMP-C2" library="rcl" package="C0603" value="10n" x="26.9875" y="33.87725"/>

Commit message: latest updates for finished hardware version 1.2
Parts:
- removed S1-E2: 10k, rcl:R0603
- added R23: 10k, rcl:R0603
- C14: value 100u -> 56u
- C16: value 100u -> 1u
- renumbered AVR-C1 to C12, AVR-C2 to C17, AVR-C3 to C11, AVR-L1 to L1, AVR-R1 to R34, D2 to D1, DISP-R1 to R1, DISP-R2 to R3, DISP-R3 to R8, DISP-R4 to R5, DISP-R5 to R4, DISP-R6 to R2, DISP-R7 to R7, DISP-R8\ to R6, IC1 to LM324, IC2 to AVR, IC3 to LDO, IC4 to OPA, LDO-C1 to C15, LDO-C2 to C2, LDO-C3 to C13, LDO-C4 to C14, LED1-R1 to R11, LED2-R1 to R18, LOET to TPSLDR, OPAMP-C1 to C4, OPAMP-C2 to C10, OPAMP-C3 to C5, OPAMP-C4 to C6, OPAMP-L1 to L2, OPAMP-R1 to R16, OPAMP-R2 to R17, OPAMP-R3 to R33, OPAMP-R4 to R19, PWR-C1 to C1, PWR-C2 to C3, PWR-R1 to R13, PWR-R2 to R10, PWR-R3 to R15, PWR-R4 to R14, PWR-R5 to R9, PWR_ENABLE to TPPWR, S1-C1 to C8, S1-R1 to R22, S2-C1 to C7, S2-R1 to R20, S2-R2 to R21, SAFETY-R1 to R35, SAFETY-R10 to R32, SAFETY-R11 to R12, SAFETY-R2 to R30, SAFETY-R3 to R31, SAFETY-R4 to R29, SAFETY-R5 to R26, SAFETY-R6 to R28, SAFETY-R7 to R24, SAFETY-R8 to R27, SAFETY-R9 to R25, SAFETY_1 to TPS1, SAFETY_2 to TPS2, SAFETY_3 to TPS3, SAFETY_C1 to C16, SAFETY_C2 to C9, TEMP_RAW to TPTEMP, U$1 to IRF
Connections:
- net BUTTON_-: now also R23.2; no longer S1-E2.2
- net N$12: now also R24.1
- net N$22: now also R23.1; no longer S1-E2.1
- net SAFETY: no longer R24.1
Routing:
- net N$12: track 10.2 -> 15.2 mm, vias 0 -> 1
- net LOETKOLBEN: track 46.1 -> 43.9 mm
- net BUTTON_-: track 55.7 -> 53.6 mm
- net N$22: track 7.29 -> 5.35 mm
- net SAFETY: track 55.1 -> 53.6 mm, vias 3 -> 2
- net ENABLE_LED_1: track 30.6 -> 29.8 mm
Other:
- board text added: "1"
- board text added: "30.04.2015 v1.2"
- board text added: "C3-C2-G"
- board text added: "DA-CL-G"
- board text added: "TX-RX-G"
- board text removed: "C3 C2 G"
- board text removed: "DA CL G"
- board text removed: "TX RX G"

Commit message: last changes
Parts:
- R12, R6: value 300 -> 330
Changed lines of the file:
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@@
 <attribute name="VALUE" x="17.78" y="32.623125" size="1.27" layer="27" rot="R90"/>
 </element>
-<element name="R6" library="rcl" package="R0603" value="300" x="14.605" y="17.8181" smashed="yes" rot="R180">
+<element name="R6" library="rcl" package="R0603" value="330" x="14.605" y="17.8181" smashed="yes" rot="R180">
 <attribute name="NAME" x="13.17625" y="18.380075" size="1.143" layer="25" font="vector" ratio="15" rot="R180"/>
 <attribute name="VALUE" x="15.24" y="19.7231" size="1.27" layer="27" rot="R180"/>
@@
 <attribute name="VALUE" x="37.2618" y="19.05" size="1.27" layer="27" rot="R180"/>
 </element>
-<element name="R12" library="rcl" package="R0603" value="300" x="36.40455" y="16.386175" smashed="yes" rot="MR180">
+<element name="R12" library="rcl" package="R0603" value="330" x="36.40455" y="16.386175" smashed="yes" rot="MR180">
 <attribute name="NAME" x="34.902775" y="18.310225" size="1.143" layer="26" font="vector" ratio="15" rot="MR180"/>
 <attribute name="VALUE" x="35.76955" y="18.291175" size="1.27" layer="28" rot="MR180"/>
