File: Hardware/v12.brd (EAGLE design)
At the start: 50 x 50 mm, 85 parts, among them J1 22-27-2081-08, J2 22-27-2031-03

Commit message: Slight changes to correct values  of some capacitors.
Parts:
- C14: value 56u -> 100u
Changed lines of the file:
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@@
 <layer number="19" name="Unrouted" color="6" fill="1" visible="yes" active="yes"/>
 <layer number="20" name="Dimension" color="15" fill="1" visible="yes" active="yes"/>
-<layer number="21" name="tPlace" color="7" fill="1" visible="no" active="yes"/>
-<layer number="22" name="bPlace" color="7" fill="1" visible="no" active="yes"/>
+<layer number="21" name="tPlace" color="7" fill="1" visible="yes" active="yes"/>
+<layer number="22" name="bPlace" color="7" fill="1" visible="yes" active="yes"/>
 <layer number="23" name="tOrigins" color="15" fill="1" visible="no" active="yes"/>
 <layer number="24" name="bOrigins" color="15" fill="1" visible="no" active="yes"/>
@@
 <attribute name="VALUE" x="9.115425" y="12.773025" size="1.27" layer="28" ratio="10" rot="MR270"/>
 </element>
-<element name="C14" library="rcl" package="E2-5" value="56u" x="4.225925" y="8.5852" smashed="yes" rot="MR0">
+<element name="C14" library="rcl" package="E2-5" value="100u" x="4.225925" y="8.5852" smashed="yes" rot="MR0">
 <attribute name="NAME" x="1.501775" y="10.188575" size="1.143" layer="26" font="vector" ratio="15" rot="MR270"/>
 <attribute name="VALUE" x="1.685925" y="6.4262" size="1.27" layer="28" ratio="10" rot="MR0"/>
