File: Hardware/v12.sch (EAGLE design)
At the start: 85 parts, among them J1 22-27-2081-08, J2 22-27-2031-03

Commit message: reworked the schematic and had to reconnect some signals in the layout. no substantial changes
Parts:
- R32: value 0 n.m. -> 1k n.m.
Connections:
- net N$32 renamed P-FET_GATE
Other:
- note added: "AVR controller"
- note added: "Buttons"
- note added: "Display (3x 7 Segment)"
- note added: "LM324 for the safety circuit"
- note added: "OpAmp for temperature measurement"
- note added: "Pin Header"
- note removed: "AVR n-Fets for the display"
- note removed: "Display 3x 7 Segment"
- note removed: "OpAmp for temp measurement (amp factor 511)"
- note removed: "two buttons"
- moved on the sheet: AVR, C1, C10, C11, C12, C13, C14, C15, C16, C17, C2, C3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
